File: tiny_bot_v2.sch (EAGLE design)
At the start: 29 parts, among them IC1 SN754410PDIP, U1 ATMEGA328P_PDIP, X1 16 MHz

Commit message: Finished routing (probably)
Parts:
- added CAPL, CAPR: 470, SparkFun-Capacitors:CAPPTH1
- LEFT_EYE, RIGHT_EYE: value LED-RGB-CC-THRUDIFFUSE -> (none); device SparkFun-LED:LED-RGB-CC-THRUDIFFUSE -> SparkFun-Connectors:M04LONGPADS
Connections:
- new net MOTOR_PWR: CAPL.2, CAPR.2, IC1.VCC2
- net GND: now also LEFT_EYE.2, RIGHT_EYE.2; no longer LEFT_EYE.CATHODE, RIGHT_EYE.CATHODE
- net N$3: now also LEFT_EYE.1; no longer LEFT_EYE.RED_CATHODE
- net N$4: now also RIGHT_EYE.1; no longer RIGHT_EYE.RED_CATHODE
- net N$5: now also LEFT_EYE.3; no longer LEFT_EYE.GREEN_CATHODE
- net N$6: now also LEFT_EYE.4; no longer LEFT_EYE.BLUE_CATHODE
- net N$7: now also RIGHT_EYE.3; no longer RIGHT_EYE.GREEN_CATHODE
- net N$8: now also RIGHT_EYE.4; no longer RIGHT_EYE.BLUE_CATHODE
- net VCC: now also CAPL.1, CAPR.1; no longer IC1.VCC2
